File: PTP_Ivan_Hodak_Project1.kicad_pcb (KiCad board)
At the start: 2 copper layers, 43 parts, among them SW1 SW_Push, SW2 SW_SPDT, U0 NE555P, U1 LM2574N-5, U2 4027, U3 4027, U4 74LS47, U5 FYS-3911BUHR-21

Commit message: PCB Update
Parts:
- removed U5: FYS-3911BUHR-21, Display_7Segment:HDSP-7401
- moved R14 67.7 mm to (90.2, 80.0)
- moved R17 64.6 mm to (87.0, 74.0)
- moved D3 63.6 mm to (139.8, 68.8), turned to 90 degrees
- moved R5 58.4 mm to (79.7, 74.0)
- moved R6 58.4 mm to (72.9, 74.0)
- moved R11 57.6 mm to (90.0, 90.8)
- moved C3 55.8 mm to (128.2, 130.2), turned to -90 degrees
- moved R16 52.7 mm to (90.0, 85.0)
- moved D5 49.6 mm to (148.0, 106.8)
- moved D2 48.2 mm to (153.0, 69.3), turned to 90 degrees
- moved R3 45.9 mm to (133.1, 67.5), turned to 180 degrees
- moved D1 44.6 mm to (153.0, 77.0), turned to 90 degrees
- moved R4 38.1 mm to (155.8, 112.1), turned to 90 degrees
- moved L1 23.5 mm to (187.5, 94.8)
- moved C1 19.5 mm to (177.0, 117.5)
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Routing:
- net +5V: track 0.00 -> 144.8 mm, vias 0 -> 4
- net GND: track 0.00 -> 84.1 mm
- net VD: track 0.00 -> 48.0 mm
- net Q0: track 0.00 -> 48.0 mm, vias 0 -> 2
- net 555: track 0.00 -> 41.0 mm, vias 0 -> 2
- net Q1: track 0.00 -> 37.1 mm, vias 0 -> 2
- net Net-(D4-K): track 0.00 -> 36.4 mm, vias 0 -> 2
- net Clock: track 0.00 -> 34.4 mm
- net Net-(U0-THR): track 0.00 -> 27.1 mm
- net Q2: track 0.00 -> 24.4 mm, vias 0 -> 2
- net Net-(U0-DIS): track 0.00 -> 20.9 mm
- net Net-(U2B-J): track 0.00 -> 20.5 mm
- net Reset: track 0.00 -> 14.6 mm
- net Net-(U2A-J): track 0.00 -> 13.1 mm
- net Net-(D5-K): track 0.00 -> 12.3 mm
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- added copper zone on B.Cu, net GND

Commit message: Update projekta
Parts:
- added U5: FYS-3911BUHR-21, Display_7Segment:HDSP-7401, F.Cu at (175.7, 102.5)
- moved R6 98.2 mm to (167.0, 102.2)
- moved R5 95.0 mm to (167.0, 111.2)
- moved R17 83.4 mm to (167.0, 97.5)
- moved R16 80.1 mm to (167.0, 106.8)
- moved R14 77.5 mm to (167.3, 87.5)
- moved C5 68.6 mm to (111.5, 109.2), turned to 90 degrees
- moved R3 56.2 mm to (151.7, 120.5), turned to 0 degrees
- moved U0 52.3 mm to (119.6, 122.6)
- moved R11 51.3 mm to (141.2, 91.2)
- moved D3 50.7 mm to (145.0, 119.2), turned to -90 degrees
- moved U4 39.8 mm to (158.6, 113.4), turned to 180 degrees
- moved SW2 36.7 mm to (117.8, 102.3)
- moved R20 34.8 mm to (121.8, 126.8)
- moved D2 31.7 mm to (127.0, 87.5)
- moved R2 31.7 mm to (138.2, 87.5)
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Routing:
- net GND: track 84.1 -> 19.4 mm
- net +5V: track 144.8 -> 191.1 mm, vias 4 -> 2
- net Net-(U4-e): track 0.00 -> 34.0 mm, vias 0 -> 2
- net Net-(U4-c): track 0.00 -> 34.0 mm, vias 0 -> 2
- net Q3: track 0.00 -> 31.0 mm, vias 0 -> 2
- net VD: track 48.0 -> 17.3 mm
- net Net-(U5-D): track 0.00 -> 30.1 mm, vias 0 -> 4
- net Net-(U4-g): track 0.00 -> 24.0 mm, vias 0 -> 2
- net Clock: track 34.4 -> 12.0 mm
- net Net-(U4-d): track 0.00 -> 21.7 mm, vias 0 -> 2
- net Q0: track 48.0 -> 69.0 mm, vias 2 -> 0
- net Net-(U4-f): track 0.00 -> 20.7 mm
- net Net-(U5-C): track 0.00 -> 18.5 mm
- net 555: track 41.0 -> 23.1 mm, vias 2 -> 6
- net Net-(U5-A): track 0.00 -> 17.0 mm
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Other:
- board outline added: 100 x 80 mm

Commit message: update
Parts:
- moved C1 5.74 mm to (188.3, 85.0)
- moved C2 5.74 mm to (199.6, 99.5)
- moved C3 5.74 mm to (116.8, 103.5)
- moved C4 5.74 mm to (200.6, 105.8)
- moved C5 5.74 mm to (111.8, 103.5)
- moved D1 5.74 mm to (123.3, 72.8)
- moved D2 5.74 mm to (127.3, 81.8)
- moved D3 5.74 mm to (145.3, 113.5)
- moved D4 5.74 mm to (187.9, 113.0)
- moved D5 5.74 mm to (161.3, 80.3)
- moved J1 5.74 mm to (176.6, 84.9)
- moved L1 5.74 mm to (194.8, 113.0)
- moved R1 5.74 mm to (134.5, 72.8)
- moved R10 5.74 mm to (134.3, 113.5)
- moved R11 5.74 mm to (141.6, 85.5)
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Routing:
- net +5V: track 191.1 -> 211.9 mm, vias 2 -> 6
- net Q3: track 31.0 -> 47.1 mm, vias 2 -> 4
- net Net-(U5-B): track 0.00 -> 16.0 mm, vias 0 -> 4
- net Net-(U5-G): track 0.00 -> 12.2 mm, vias 0 -> 2
- net Net-(U5-F): track 0.00 -> 11.8 mm, vias 0 -> 2
- net GND: track 19.4 -> 27.6 mm, vias 0 -> 2
- net Net-(R13-Pad1): track 0.00 -> 6.50 mm
- net Net-(U4-g): track 24.0 -> 17.6 mm
- net Net-(U4-BI): track 13.8 -> 19.7 mm, vias 0 -> 2
- net Net-(U4-f): track 20.7 -> 26.3 mm
- net Net-(U2B-J): track 9.04 -> 11.6 mm
- net Net-(U2A-J): track 11.2 -> 13.8 mm
- net Net-(U5-A): track 17.0 -> 19.3 mm
Other:
- board text added: "Projekt PTP - Ivan Hodak"
